File: RP-Pico-KiCad/Turing-Circuit/Turing-Circuit.kicad_sch (KiCad schematic)
At the start: 14 parts

Commit message: Circuit Finished
Project circuit in KiCad
Parts:
- added R6, R7: R, symbol Device:R
Connections:
- net GP14: now reaches R4.1
- net GP14: no longer RP-Pico1. (VSYS)
- net GP23: now reaches 7-Segment1. (g)
- net GP23: no longer RP-Pico1. (VSYS)
- net GP15: now reaches R5.1
- net GP15: no longer RP-Pico1. (VSYS)
- net GND: now reaches D1.1 (K), D2.1 (K), D3.1 (K), D4.1 (K), D5.1 (K)
- net GND: now also 7-Segment1. (g), button_left.2, button_right.2; no longer RP-Pico1. (VSYS)
- net GP11: now reaches R1.2
- net GP11: no longer RP-Pico1. (VSYS)
- net GP12: now reaches R2.2
- net GP12: no longer RP-Pico1. (VSYS)
- net GP13: now reaches R3.1
- net GP13: no longer RP-Pico1. (VSYS)
- net GP2: now reaches button_right.4 (A)
- net GP2: now also R6.2
- net GP3: now reaches button_left.4 (A)
- net GP3: now also R7.2
- new net GP16: 7-Segment1. (g)
- new net GP17: 7-Segment1. (g)
- new net GP18: 7-Segment1. (g)
- new net GP19: 7-Segment1. (g)
- new net GP20: 7-Segment1. (g)
- new net GP21: 7-Segment1. (g)
- new net GP22: 7-Segment1. (g)
- new net VCC: R6.1, R7.1
- now unconnected: RP-Pico1. (VSYS), RP-Pico1. (VSYS), RP-Pico1. (VSYS), RP-Pico1. (VSYS), RP-Pico1. (VSYS), RP-Pico1. (VSYS), RP-Pico1. (VSYS)
Other:
- moved on the sheet: button_left, button_right

Commit message: bugfixes and schematic
adding ciruit schematic for project
bux fixes
Parts:
- added R10, R11, R12, R13, R14, R16, R17, R8, R9: R, symbol Device:R
Connections:
- net GND: now also R12.2; no longer 7-Segment1. (g)
- net GP16: now also R9.2; no longer 7-Segment1. (g)
- net GP17: now also R8.2; no longer 7-Segment1. (g)
- net GP18: now also R14.2; no longer 7-Segment1. (g)
- net GP19: now also R16.2; no longer 7-Segment1. (g)
- net GP20: now also R17.2; no longer 7-Segment1. (g)
- net GP21: now also R11.2; no longer 7-Segment1. (g)
- net GP22: now also R10.2; no longer 7-Segment1. (g)
- net GP23: now also R13.2; no longer 7-Segment1. (g)
- new net: 7-Segment1. (g), R12.1
- new net: 7-Segment1. (g), R10.1
- new net: 7-Segment1. (g), R8.1
- new net: 7-Segment1. (g), R13.1
- new net: 7-Segment1. (g), R16.1
- new net: 7-Segment1. (g), R17.1
- new net: 7-Segment1. (g), R9.1
- new net: 7-Segment1. (g), R14.1
- new net: 7-Segment1. (g), R11.1
Other:
- moved on the sheet: button_left, button_right
